File: KiCad/LoRaWX01.kicad_pcb (KiCad board)
At the start: 2 copper layers, 26 parts, among them J1 BATT, J10 DEBUG, J2 SOLAR, J3 + input, J4 GND, J5 + output, J6 GND, J7 W_SONDA, J8 ANT-433, U1 LF33_TO252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

Commit message: zmeny v napajeni bme280
Parts:
- added D1: LED, Resistor_THT:R_Axial_DIN0204_L3.6mm_D1.6mm_P5.08mm_Vertical, F.Cu at (119.3, 93.0)
- C4: value 500uF -> 50uF
- J2: value SOLAR -> SOLAR 5,5-6V
- J7: moved to F.Cu
- R1: value 99K -> 91K18
- R2: value 10K -> 10K09
- moved J3 15.9 mm to (148.7, 108.3)
- moved J4 15.8 mm to (132.8, 108.5)
- moved J7 4.59 mm to (121.2, 106.3), turned to 180 degrees
- moved J2 2.41 mm to (133.0, 116.3), turned to 90 degrees
- renumbered Rain to J11
Connections:
- C3 pad 1: Net-(U2-Pad20) -> Net-(C3-Pad1)
- C4 pad 1: Net-(U2-Pad20) -> Net-(C3-Pad1)
- J7 pad 2: Net-(R6-Pad2) -> GND
- J7 pad 3: GND -> Net-(D1-Pad2)
- R3 pad 1: Net-(U2-Pad20) -> Net-(C3-Pad1)
- R6 pad 1: Net-(U2-Pad20) -> Net-(C3-Pad1)
- R6 pad 2: Net-(R6-Pad2) -> Net-(D1-Pad2)
- R7 pad 1: Net-(U2-Pad20) -> Net-(C3-Pad1)
- R8 pad 1: Net-(U2-Pad20) -> Net-(C3-Pad1)
- U1 pad 3: Net-(U2-Pad20) -> Net-(C3-Pad1)
- U2 pad 14: unconnected-(U2-Pad14) -> srdce
- U2 pad 15: unconnected-(U2-Pad15) -> Net-(U2-Pad15)
- U2 pad 20: Net-(U2-Pad20) -> Net-(C3-Pad1)
- U2 pad 4: Net-(R6-Pad2) -> Net-(D1-Pad2)
- U2 pad 7: Net-(U2-Pad20) -> Net-(C3-Pad1)
- U3 pad 1: Net-(U2-Pad20) -> Net-(U2-Pad15)
- U4 pad 13: Net-(U2-Pad20) -> Net-(C3-Pad1)
Routing:
- net Net-(U2-Pad20): track 154.1 -> 0.00 mm, vias 2 -> 0
- net Net-(C3-Pad1): track 0.00 -> 153.9 mm, vias 0 -> 2
- net GND: track 615.9 -> 565.8 mm
- net Net-(D1-Pad2): track 0.00 -> 45.5 mm
- net Net-(U2-Pad15): track 0.00 -> 42.7 mm, vias 0 -> 2
- net Net-(R6-Pad2): track 37.7 -> 0.00 mm
- net Net-(J2-Pad2): track 6.53 -> 16.5 mm
- net Net-(R1-Pad2): track 43.2 -> 40.9 mm
Other:
- board text added: "2021/09"
- board text added: "OK1FET 2021/09 v2"
- board text removed: "2021/03"
- board text removed: "OK1FET 2021/03 v1"
